File: MAX2769FT2232H.kicad_pcb (KiCad board)
At the start: 4 copper layers, 88.9 x 50.8 mm, 99 parts, among them J1 Conn_Coaxial, J2 USB_A, J3 RF_Shield_One_Piece, J4 Conn_Coaxial, U1 MAX2769ETI+T, U10 74LVC374, U11 74HC2G04, U2 TPS717285DCKR, U3 TPS717285DCKR, U4 NCP164CSN330T1G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

Commit message: Added Note concerning voltage regulator caps
Other:
- board text added: "FT2232H<->MAX2769"
