File: MAX2769FT2232H.sch (KiCad schematic (older format))
At the start: 99 parts, among them J1 Conn_Coaxial, J2 USB_A, J3 RF_Shield_One_Piece, J4 Conn_Coaxial, U1 MAX2769ETI+T, U10 74LVC374, U11 74HC2G04, U2 TPS717285DCKR, U3 TPS717285DCKR, U4 NCP164CSN330T1G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

Commit message: Added Note concerning voltage regulator caps
Other:
- note added: "MAX8510: C22<=10 nF, C47<=NC\nTI717: C47<=10 nF, C22<=NC"
- note added: "MAX8510: C26<=10 nF, C48<=NC\nTI717: C48<=10 nF, C26<=NC"
Changed lines of the file:
@@
 	1    0    0    -1
 $EndComp
+Text Notes 14350 1550 0    50   ~ 0
+MAX8510: C26<=10 nF, C48<=NC\nTI717:    C48<=10 nF, C26<=NC
 Wire Bus Line
 	6550 600  12550 600
@@
 Wire Bus Line
 	9000 1800 9000 4300
+Text Notes 14350 4450 0    50   ~ 0
+MAX8510: C22<=10 nF, C47<=NC\nTI717:    C47<=10 nF, C22<=NC
 $EndSCHEMATC
